File: mcu.kicad_sch (KiCad schematic)
At the start: 16 parts, among them IC1 STM32C542CCT6, J8 Conn_02x05_Odd_Even, SW1 SW_Push, Y3 ECS-120-18-33-JGN-TR

Commit message: changes?
Parts:
- Y3: value ECS-120-18-33-JGN-TR -> ECS-400-18-33-JGN-TR
Changed lines of the file:
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@@
 			)
 		)
-		(property "Value" "ECS-120-18-33-JGN-TR"
+		(property "Value" "ECS-400-18-33-JGN-TR"
 			(at 240.03 105.41 0)
 			(show_name no)
