File: mcu.kicad_sch (KiCad schematic)
At the start: 16 parts, among them IC1 STM32C542CCT6, J8 Conn_02x05_Odd_Even, SW1 SW_Push, Y3 ECS-400-18-33-JGN-TR

Commit message: In progress, changed stdby
Connections:
- net STBY_STM: no longer names the net of IC1.11 (PA1)
- no-connect marks 30 -> 31
Changed lines of the file:
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@@
+	)
+	(no_connect
+		(at 156.21 81.28)
 	)
 	(no_connect
@@
 		(pts
 			(xy 227.33 24.13) (xy 237.49 24.13)
-		)
-		(stroke
-			(width 0)
-			(type default)
-		)
-	)
-	(wire
-		(pts
-			(xy 154.94 81.28) (xy 156.21 81.28)
 		)
 		(stroke
@@
 			)
 		)
-	)
-	(global_label "STBY_STM"
-		(shape input)
-		(at 154.94 81.28 180)
-		(fields_autoplaced yes)
-		(effects
-			(font
-				(size 1.016 1.016)
-			)
-			(justify right)
-		)
-		(property "Intersheetrefs" "${INTERSHEET_REFS}"
-			(at 145.7698 81.28 0)
-			(hide yes)
-			(show_name no)
-			(do_not_autoplace no)
-			(effects
-				(font
-					(size 1.27 1.27)
-				)
-				(justify right)
-			)
-		)

Commit message: Relatively final changes
Parts:
- removed IC1: STM32C542CCT6, QFP50P900X900X160-48N, symbol STM32C542CCT6:STM32C542CCT6
- added U7: STM32C542CCT6, LQFP48-7X7, symbol 2026-09-19_00-19-05:STM32C542CCT6
- C11: value 0.1u -> 100n
- C14, C15: value 27pF -> 27p
Connections:
- net +3.3V: now also J8.1 (Pin_1), U7.24 (VDD), U7.36 (VDD), U7.48 (VDD), U7.9 (VREF+); no longer J8.7 (Pin_7), J8.8 (Pin_8)
- net GND: now also J8.3 (Pin_3), J8.9 (Pin_9), U7.23 (VSS), U7.35 (VSS), U7.47 (VSS), U7.8 (VREF-); no longer J8.6 (Pin_6)
- net GPIO_ALERT: now also U7.41 (PB5)
- net I2C_SCL_STM: now also U7.42 (PB6)
- net I2C_SDA_STM: now also U7.43 (PB7)
- net NRST: now also J8.10 (Pin_10), U7.7 (NRST); no longer J8.1 (Pin_1)
- net OSC_IN_STM: now also U7.5 (PH0-OSC_IN)
- net OSC_OUT_STM: now also U7.6 (PH1-OSC_OUT)
- net STM_LED: now also U7.29 (PA8)
- net SWCLK: now also J8.4 (Pin_4), U7.37 (PA14); no longer J8.2 (Pin_2)
- net SYS_SWDIO: now also J8.2 (Pin_2), U7.34 (PA13); no longer J8.4 (Pin_4)
- net V_CAP: now also U7.22 (VCAP)
- new net CS_PI: U7.17 (PA7)
- new net MISO: U7.16 (PA6)
- new net MOSI: U7.14 (PA4)
- new net SCLK: U7.15 (PA5)
- new net STM_CAN_RX: U7.32 (PA11)
- new net STM_CAN_TX: U7.33 (PA12)
- new net USART1_RX: U7.31 (PA10)
- new net USART1_TX: U7.30 (PA9)
- no-connect marks 31 -> 25
Other:
- note added: "Left 3 all for VDD_1 2 3. 4.7u parallel with all three VDD cap to ground Second right to VREF+ Right to VCap"
- note added: "STM32 MCU Pinout"
- note removed: "C16 C17 C18 all for VDD_1 2 3. 4.7u parallel with all three VDD cap to ground C14 to VREF+ C15 to VCap"
- moved on the sheet: C11, C14, C15, C20, C21, C22, C23, C24, C25, J8, R2, R3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

Commit message: Some minor changes
Parts:
- removed J8: Conn_02x05_Odd_Even, Oscillator:Oscillator_SMD_ECS_2520MV-xxx-xx-4Pin_2.5x2.0mm, symbol Connector_Generic:Conn_02x05_Odd_Even
- removed R2, R3: 4.7k, symbol Device:R_Small_US
- added J9: Conn_01x05, symbol Connector_Generic:Conn_01x05
- added R26, R27: 4.7k, symbol Device:R_US
Connections:
- net +3.3V: now also J9.1 (Pin_1), R26.2, R27.2
- net GND: now also J9.5 (Pin_5)
- net I2C_SCL_STM: now also R26.1
- net I2C_SDA_STM: now also R27.1
- net NRST: now also J9.4 (Pin_4)
- net SWCLK: now also J9.3 (Pin_3)
- net SYS_SWDIO: now also J9.2 (Pin_2)
- net CS_PI renamed CS_STM
- net GPIO_ALERT renamed ALERT_5.1V
- no-connect marks 25 -> 22
Other:
- note removed: "I2C Pullups Place close to STM"
- moved on the sheet: U7

Commit message: updated footprints
Parts:
- U7: footprint LQFP48-7X7 -> (none)
Changed lines of the file:
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@@
 			)
 		)
-		(property "Footprint" "LQFP48-7X7"
+		(property "Footprint" ""
 			(at 39.37 38.1 0)
 			(hide yes)

Commit message: added footprints
Parts:
- C11, C14, C15, C20, C21, C22, C23, C24, C25: footprint (none) -> Capacitor_SMD:C_0603_1608Metric_Pad1.08x0.95mm_HandSolder
- J9: footprint (none) -> Connector_PinHeader_2.54mm:PinHeader_1x05_P2.54mm_Horizontal
- R26, R27: footprint (none) -> Resistor_SMD:R_0603_1608Metric_Pad0.98x0.95mm_HandSolder
Changed lines of the file:
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@@
+			)
+		)
+		(property "digikey" ""
+			(at 166.37 134.62 90)
+			(hide yes)
+			(show_name no)
+			(do_not_autoplace no)
+			(effects
+				(font
+					(size 1.27 1.27)
+				)
 			)
 		)
@@
 			)
 		)
+		(property "digikey" ""
+			(at 232.41 78.74 0)
+			(hide yes)
+			(show_name no)
+			(do_not_autoplace no)
+			(effects
+				(font
+					(size 1.27 1.27)
+				)
+			)
+		)
 		(pin "1"
 		)
@@
 			)
 		)
-		(property "Footprint" ""
+		(property "Footprint" "Capacitor_SMD:C_0603_1608Metric_Pad1.08x0.95mm_HandSolder"
 			(at 163.5252 40.64 0)
 			(hide yes)
@@
 		)
 		(property "Description" "Unpolarized capacitor"
+			(at 162.56 36.83 0)
+			(hide yes)
+			(show_name no)
+			(do_not_autoplace no)
+			(effects
+				(font
+					(size 1.27 1.27)
+				)
+			)
+		)
+		(property "digikey" ""
 			(at 162.56 36.83 0)
 			(hide yes)
@@
 			)
 		)
+		(property "digikey" ""
+			(at 179.07 121.92 0)
+			(hide yes)
+			(show_name no)
+			(do_not_autoplace no)
+			(effects
+				(font
+					(size 1.27 1.27)
+				)
+			)
+		)
 		(pin "2"
 		)
@@
 			)
 		)
-		(property "Footprint" ""
+		(property "Footprint" "Resistor_SMD:R_0603_1608Metric_Pad0.98x0.95mm_HandSolder"
 			(at 118.364 44.196 90)
 			(hide yes)
@@
 			)
 		)
+		(property "digikey" ""
+			(at 119.38 44.45 0)
+			(hide yes)
+			(show_name no)
+			(do_not_autoplace no)
+			(effects
+				(font
+					(size 1.27 1.27)
+				)
+			)
+		)
 		(pin "2"
 		)
@@
 			)
 		)
-		(property "Footprint" ""
+		(property "Footprint" "Capacitor_SMD:C_0603_1608Metric_Pad1.08x0.95mm_HandSolder"
 			(at 192.7352 40.64 0)
 			(hide yes)
@@
 			)
 		)
+		(property "digikey" ""
+			(at 191.77 36.83 0)
+			(hide yes)
+			(show_name no)
+			(do_not_autoplace no)
+			(effects
+				(font
+					(size 1.27 1.27)
+				)
+			)
+		)
 		(pin "1"
 		)
@@
 			)
 		)
-		(property "Footprint" ""
+		(property "Footprint" "Capacitor_SMD:C_0603_1608Metric_Pad1.08x0.95mm_HandSolder"
 			(at 183.8452 40.64 0)
 			(hide yes)
@@
 		)
 		(property "Description" "Unpolarized capacitor"
+			(at 182.88 36.83 0)
+			(hide yes)
+			(show_name no)
+			(do_not_autoplace no)
+			(effects
+				(font
+					(size 1.27 1.27)
+				)
+			)
+		)
+		(property "digikey" ""
 			(at 182.88 36.83 0)
 			(hide yes)
@@
 			)
 		)
-		(property "Footprint" ""
+		(property "Footprint" "Capacitor_SMD:C_0603_1608Metric_Pad1.08x0.95mm_HandSolder"
 			(at 208.5848 77.47 0)
 			(hide yes)
@@
 		)
 		(property "Description" "Unpolarized capacitor"
+			(at 209.55 81.28 0)
+			(hide yes)
+			(show_name no)
+			(do_not_autoplace no)
+			(effects
+				(font
+					(size 1.27 1.27)
+				)
+			)
+		)
+		(property "digikey" ""
 			(at 209.55 81.28 0)
 			(hide yes)
@@
 			)
 		)
-		(property "Footprint" ""
+		(property "Footprint" "Capacitor_SMD:C_0603_1608Metric_Pad1.08x0.95mm_HandSolder"
 			(at 213.0552 40.64 0)
 			(hide yes)
@@
 		)
 		(property "Description" "Unpolarized capacitor"
+			(at 212.09 36.83 0)
+			(hide yes)
+			(show_name no)
+			(do_not_autoplace no)
+			(effects
+				(font
+					(size 1.27 1.27)
+				)
+			)
+		)
+		(property "digikey" ""
 			(at 212.09 36.83 0)
 			(hide yes)
@@
 			)
 		)
-		(property "Footprint" ""
+		(property "Footprint" "Connector_PinHeader_2.54mm:PinHeader_1x05_P2.54mm_Horizontal"
 			(at 72.39 133.35 0)
 			(hide yes)
@@
 		)
 		(property "Description" "Generic connector, single row, 01x05, script generated (kicad-library-utils/schlib/autogen/connector/)"
+			(at 72.39 133.35 0)
+			(hide yes)
+			(show_name no)
+			(do_not_autoplace no)
+			(effects
+				(font
+					(size 1.27 1.27)
+				)
+			)
+		)
+		(property "digikey" ""
 			(at 72.39 133.35 0)
 			(hide yes)
@@
 			)
 		)
-		(property "Footprint" ""
+		(property "Footprint" "Capacitor_SMD:C_0603_1608Metric_Pad1.08x0.95mm_HandSolder"
 			(at 180.0352 137.16 0)
 			(hide yes)
@@
 		)
 		(property "Description" "Unpolarized capacitor"
+			(at 179.07 133.35 0)
+			(hide yes)
+			(show_name no)
+			(do_not_autoplace no)
+			(effects
+				(font
+					(size 1.27 1.27)
+				)
+			)
+		)
+		(property "digikey" ""
 			(at 179.07 133.35 0)
 			(hide yes)
@@
 			)
 		)
+		(property "digikey" ""
+			(at 39.37 38.1 0)
+			(hide yes)
+			(show_name no)
+			(do_not_autoplace no)
+			(effects
+				(font
+					(size 1.27 1.27)
+				)
+			)
+		)
 		(pin "23"
 		)
@@
 			)
 		)
-		(property "Footprint" ""
+		(property "Footprint" "Capacitor_SMD:C_0603_1608Metric_Pad1.08x0.95mm_HandSolder"
 			(at 261.3152 85.09 0)
 			(hide yes)
@@
 			)
 		)
+		(property "digikey" ""
+			(at 260.35 81.28 0)
+			(hide yes)
+			(show_name no)
+			(do_not_autoplace no)
+			(effects
+				(font
+					(size 1.27 1.27)
+				)
+			)
+		)
 		(pin "1"
 		)
@@
 			)
 		)
-		(property "Footprint" ""
+		(property "Footprint" "Capacitor_SMD:C_0603_1608Metric_Pad1.08x0.95mm_HandSolder"
 			(at 202.8952 40.64 0)
 			(hide yes)
@@
 			)
 		)
+		(property "digikey" ""
+			(at 201.93 36.83 0)
+			(hide yes)
+			(show_name no)
+			(do_not_autoplace no)
+			(effects
+				(font
+					(size 1.27 1.27)
+				)
+			)
+		)
 		(pin "1"
 		)
@@
 			)
 		)
-		(property "Footprint" ""
+		(property "Footprint" "Capacitor_SMD:C_0603_1608Metric_Pad1.08x0.95mm_HandSolder"
 			(at 173.6852 40.64 0)
 			(hide yes)
@@
 			)
 		)
+		(property "digikey" ""
+			(at 172.72 36.83 0)
+			(hide yes)
+			(show_name no)
+			(do_not_autoplace no)
+			(effects
+				(font
+					(size 1.27 1.27)
+				)
+			)
+		)
 		(pin "1"
 		)
@@
 			)
 		)
-		(property "Footprint" ""
+		(property "Footprint" "Resistor_SMD:R_0603_1608Metric_Pad0.98x0.95mm_HandSolder"
 			(at 125.984 44.196 90)
 			(hide yes)
@@
 			(at 127 44.45 0)
 			(hide yes)
+			(show_name no)
+			(do_not_autoplace no)
+			(effects
+				(font
+					(size 1.27 1.27)
+				)
+			)
+		)
+		(property "digikey" ""
+			(at 127 44.45 0)
+			(hide yes)

Commit message: almost done with footprints
Parts:
- U7: footprint (none) -> rov_STM_footprint:LQFP48-7X7-M
Changed lines of the file:
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@@
 			)
 		)
-		(property "Footprint" ""
+		(property "Footprint" "rov_STM_footprint:LQFP48-7X7-M"
 			(at 39.37 38.1 0)
 			(hide yes)

Commit message: done with footprints! one more thing for leak sensors
Parts:
- J9: footprint Connector_PinHeader_2.54mm:PinHeader_1x05_P2.54mm_Horizontal -> Connector_PinHeader_2.54mm:PinHeader_1x05_P2.54mm_Vertical
- R5: footprint Resistor_THT:R_Array_SIP4 -> Resistor_SMD:R_0603_1608Metric_Pad0.98x0.95mm_HandSolder
- SW1: footprint Button_Switch_THT:SW_NKK_GW12LJP -> rov_switch_FSM2JMTR:SW_FSM2JMTR_TEC-M
- Y3: footprint ECS-120-18-33-JGN-TR:XTAL_ECS-120-18-33-JGN-TR -> rov_ECS_400_18_33_JGN_TR:XTAL_ECS-400-18-33-JGN-TR
Changed lines of the file:
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@@
 			)
 		)
-		(property "Footprint" "Button_Switch_THT:SW_NKK_GW12LJP"
+		(property "Footprint" "rov_switch_FSM2JMTR:SW_FSM2JMTR_TEC-M"
 			(at 161.29 134.62 0)
 			(hide yes)
@@
 			)
 		)
-		(property "Footprint" "ECS-120-18-33-JGN-TR:XTAL_ECS-120-18-33-JGN-TR"
+		(property "Footprint" "rov_ECS_400_18_33_JGN_TR:XTAL_ECS-400-18-33-JGN-TR"
 			(at 232.41 78.74 0)
 			(hide yes)
@@
 			)
 		)
-		(property "Footprint" "Resistor_THT:R_Array_SIP4"
+		(property "Footprint" "Resistor_SMD:R_0603_1608Metric_Pad0.98x0.95mm_HandSolder"
 			(at 180.086 122.174 90)
 			(hide yes)
@@
 			)
 		)
-		(property "Footprint" "Connector_PinHeader_2.54mm:PinHeader_1x05_P2.54mm_Horizontal"
+		(property "Footprint" "Connector_PinHeader_2.54mm:PinHeader_1x05_P2.54mm_Vertical"
 			(at 72.39 133.35 0)
 			(hide yes)

Commit message: footprints COMPLETELY DONE
Parts:
- added D5: LED, LED_SMD:LED_0805_2012Metric_Pad1.15x1.40mm_HandSolder, symbol Device:LED
- added J10: Conn_01x03, Connector_PinHeader_2.54mm:PinHeader_1x03_P2.54mm_Vertical, symbol Connector_Generic:Conn_01x03
- added J11: Conn_01x06, Connector_PinHeader_2.54mm:PinHeader_1x06_P2.54mm_Vertical, symbol Connector_Generic:Conn_01x06
- added J12, J13, J14, J15: Conn_01x03, Connector_JST:JST_GH_BM02B-GHS-TBT_1x02-1MP_P1.25mm_Vertical, symbol Connector_Generic:Conn_01x03
- added Q1: MMBT3906, Package_TO_SOT_SMD:SOT-23-3, symbol Transistor_BJT:2N3905
- added R14, R2: 1K, Resistor_SMD:R_0603_1608Metric_Pad0.98x0.95mm_HandSolder, symbol Device:R_US
- added R15: 240, Resistor_SMD:R_0603_1608Metric_Pad0.98x0.95mm_HandSolder, symbol Device:R_US
- added R3: 27K, Resistor_SMD:R_0603_1608Metric_Pad0.98x0.95mm_HandSolder, symbol Device:R_US
- C14, C15: value 27p -> 10p
- Y3: value ECS-400-18-33-JGN-TR -> ECS-240-8-37B-CKY_TR; footprint rov_ECS_400_18_33_JGN_TR:XTAL_ECS-400-18-33-JGN-TR -> rov_ECS-240-8-37B-CKY-TR:XTAL_ECS-160-9-37-CKM-TR
Connections:
- net GND: now also D5.1 (K), J10.1 (Pin_1), J12.1 (Pin_1), J12.2 (Pin_2), J13.1 (Pin_1), J13.2 (Pin_2), J14.1 (Pin_1), J14.2 (Pin_2), J15.1 (Pin_1), J15.2 (Pin_2), R14.2
- net LEAK_STM: now reaches U7.10 (PA0)
- net LEAK_STM: now also J10.3 (Pin_3), Q1.3 (C), R14.1, R15.1
- net at U7.13 (PA3): now also J11.6 (Pin_6)
- net at U7.25 (PB12): now also J11.5 (Pin_5)
- net at U7.26 (PB13): now also J11.4 (Pin_4)
- net at U7.27 (PB14): now also J11.3 (Pin_3)
- net at U7.45 (PB8): now also J11.2 (Pin_2)
- net at U7.46 (PB9): now also J11.1 (Pin_1)
- new net: D5.2 (A), R15.2
- new net: Q1.2 (B), R2.2, R3.2
- new net PROBE: J12.3 (Pin_3), J13.3 (Pin_3), J14.3 (Pin_3), J15.3 (Pin_3), R2.1
- new net VCC: J10.2 (Pin_2), Q1.1 (E), R3.1
- no-connect marks 22 -> 14
Other:
- moved on the sheet: J9, U7
