File: can.kicad_sch (KiCad schematic)
At the start: 14 parts, among them U4 TCAN1044VDRQ1, U5 MCP2518FDT-E/QBB, U6 TCAN1044VDRQ1, Y1 ECS-120-18-33-JGN-TR

Commit message: changes?
Parts:
- Y1: value ECS-120-18-33-JGN-TR -> ECS-400-18-33-JGN-TR
Changed lines of the file:
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@@
+		)
+	)
+	(hierarchical_label "g"
+		(shape input)
+		(at 179.07 125.73 0)
+		(effects
+			(font
+				(size 1.27 1.27)
+			)
+			(justify left)
 		)
 	)
@@
 			)
 		)
-		(property "Value" "ECS-120-18-33-JGN-TR"
+		(property "Value" "ECS-400-18-33-JGN-TR"
 			(at 60.96 86.36 0)
 			(show_name no)

Commit message: In progress, changed stdby
Parts:
- added TP5: TestPoint, symbol Connector:TestPoint
- C17: value 0.1u -> 4.7uF
Connections:
- net STBY_MCP is gone; now on net GND: U4.8 (STB)
- net STBY_STM is gone; now on net GND: U6.8 (STB)
- net GND: now also U5.9 (*INT0/GPIO0/XSTBY)
- net INT_PI: now also TP5.1
- no-connect marks 2 -> 1
Other:
- moved on the sheet: C3, C4, C6, U5, Y1

Commit message: Relatively final changes
Parts:
- removed TP5: TestPoint, symbol Connector:TestPoint
- added C28: 1u, symbol Device:C
- added R11: 10K, symbol Device:R_US
- added TP10, TP11, TP8: TestPoint, symbol Connector:TestPoint
- C12, C13, C7, C8: value 100nF -> 100n
- C17: value 4.7uF -> 4.7n
- C3, C4: value 27pF -> 27p
- C6: value 0.1u -> 100n
Connections:
- net +3.3V: now also C28.1, R11.1
- net CS_PI: now also R11.2
- net GND: now also C28.2; no longer U5.9 (*INT0/GPIO0/XSTBY)
- net at U5.3 (CLKO/SOF): now also TP8.1
- net at U5.8 (*INT1/GPIO1): now also TP11.1
- net +5V renamed +5.1V
- net RXDSTM renamed STM_CAN_RX
- net TXDSTM renamed STM_CAN_TX
- new net: TP10.1, U5.9 (*INT0/GPIO0/XSTBY)
- no-connect marks 1 -> 0
Other:
- moved on the sheet: C12, C13, C17, C3, C4, C6, C7, C8, R12, R13, U4, U5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

Commit message: Some minor changes
Changed lines of the file:
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@@
 		(effects
 			(font
-				(size 1.016 1.016)
-			)
-			(justify right)
-		)
-		(property "Intersheetrefs" "${INTERSHEET_REFS}"
-			(at 147.5478 40.64 0)
+				(size 1.27 1.27)
+			)
+			(justify right)
+		)
+		(property "Intersheetrefs" "${INTERSHEET_REFS}"
+			(at 144.7471 40.64 0)
 			(hide yes)
 			(show_name no)
@@
 		(effects
 			(font
-				(size 1.016 1.016)
-			)
-			(justify right)
-		)
-		(property "Intersheetrefs" "${INTERSHEET_REFS}"
-			(at 59.5791 43.18 0)
+				(size 1.27 1.27)
+			)
+			(justify right)
+		)
+		(property "Intersheetrefs" "${INTERSHEET_REFS}"
+			(at 57.9637 43.18 0)
 			(hide yes)
 			(show_name no)
@@
 		(effects
 			(font
-				(size 1.016 1.016)
-			)
-			(justify left)
-		)
-		(property "Intersheetrefs" "${INTERSHEET_REFS}"
-			(at 222.1069 40.64 0)
+				(size 1.27 1.27)
+			)
+			(justify left)
+		)
+		(property "Intersheetrefs" "${INTERSHEET_REFS}"
+			(at 225.2462 40.64 0)
 			(hide yes)
 			(show_name no)
@@
 		(effects
 			(font
-				(size 1.016 1.016)
-			)
-			(justify right)
-		)
-		(property "Intersheetrefs" "${INTERSHEET_REFS}"
-			(at 61.1878 48.26 0)
+				(size 1.27 1.27)
+			)
+			(justify right)
+		)
+		(property "Intersheetrefs" "${INTERSHEET_REFS}"
+			(at 58.3871 48.26 0)
 			(hide yes)
 			(show_name no)
@@
 		(effects
 			(font
-				(size 1.016 1.016)
-			)
-			(justify left)
-		)
-		(property "Intersheetrefs" "${INTERSHEET_REFS}"
-			(at 123.3855 45.72 0)
+				(size 1.27 1.27)
+			)
+			(justify left)
+		)
+		(property "Intersheetrefs" "${INTERSHEET_REFS}"
+			(at 125.3396 45.72 0)
 			(hide yes)
 			(show_name no)
@@
 		(effects
 			(font
-				(size 1.016 1.016)
-			)
-			(justify left)
-		)
-		(property "Intersheetrefs" "${INTERSHEET_REFS}"
-			(at 127.1109 38.1 0)
+				(size 1.27 1.27)
+			)
+			(justify left)
+		)
+		(property "Intersheetrefs" "${INTERSHEET_REFS}"
+			(at 129.9962 38.1 0)
 			(hide yes)
 			(show_name no)
@@
 		(effects
 			(font
-				(size 1.016 1.016)
-			)
-			(justify left)
-		)
-		(property "Intersheetrefs" "${INTERSHEET_REFS}"
-			(at 126.869 35.56 0)
+				(size 1.27 1.27)
+			)
+			(justify left)
+		)
+		(property "Intersheetrefs" "${INTERSHEET_REFS}"
+			(at 129.6938 35.56 0)
 			(hide yes)
 			(show_name no)
@@
 		(effects
 			(font
-				(size 1.016 1.016)
-			)
-			(justify left)
-		)
-		(property "Intersheetrefs" "${INTERSHEET_REFS}"
-			(at 140.7422 40.64 0)
+				(size 1.27 1.27)
+			)
+			(justify left)
+		)
+		(property "Intersheetrefs" "${INTERSHEET_REFS}"
+			(at 142.2729 40.64 0)
 			(hide yes)
 			(show_name no)
@@
 		(effects
 			(font
-				(size 1.016 1.016)
-			)
-			(justify left)
-		)
-		(property "Intersheetrefs" "${INTERSHEET_REFS}"
-			(at 123.3855 43.18 0)
+				(size 1.27 1.27)
+			)
+			(justify left)
+		)
+		(property "Intersheetrefs" "${INTERSHEET_REFS}"
+			(at 125.3396 43.18 0)
 			(hide yes)
 			(show_name no)
@@
 		(effects
 			(font
-				(size 1.016 1.016)
-			)
-			(justify left)
-		)
-		(property "Intersheetrefs" "${INTERSHEET_REFS}"
-			(at 123.5307 48.26 0)
+				(size 1.27 1.27)
+			)
+			(justify left)
+		)
+		(property "Intersheetrefs" "${INTERSHEET_REFS}"
+			(at 125.521 48.26 0)
 			(hide yes)
 			(show_name no)
@@
 		(effects
 			(font
-				(size 1.016 1.016)
-			)
-			(justify right)
-		)
-		(property "Intersheetrefs" "${INTERSHEET_REFS}"
-			(at 59.8331 45.72 0)
-			(hide yes)
-			(show_name no)
+				(size 1.27 1.27)
+			)
+			(justify right)
+		)
+		(property "Intersheetrefs" "${INTERSHEET_REFS}"
+			(at 56.6938 45.72 0)
+			(hide yes)
+			(show_name no)

Commit message: updated footprints
Parts:
- U4, U6: footprint D0008A-IPC_A -> (none)
- U5: footprint VDFN14_QBB_MCH -> (none)
Changed lines of the file:
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@@
 			)
 		)
-		(property "Footprint" "D0008A-IPC_A"
+		(property "Footprint" ""
 			(at 111.76 130.81 0)
 			(hide yes)
@@
 			)
 		)
-		(property "Footprint" "VDFN14_QBB_MCH"
+		(property "Footprint" ""
 			(at 72.39 35.56 0)
 			(hide yes)
@@
 			)
 		)
-		(property "Footprint" "D0008A-IPC_A"
+		(property "Footprint" ""
 			(at 111.76 86.36 0)
 			(hide yes)

Commit message: added footprints
Parts:
- C12, C13, C17, C28, C3, C4, C6, C7, C8: footprint (none) -> Capacitor_SMD:C_0603_1608Metric_Pad1.08x0.95mm_HandSolder
- R11, R12, R13: footprint (none) -> Resistor_SMD:R_0603_1608Metric_Pad0.98x0.95mm_HandSolder
- TP10, TP11, TP8: footprint (none) -> TestPoint:TestPoint_Pad_D1.5mm
- U5: footprint (none) -> rov_MCP_footprint:VDFN14_QBB_MCH-M

Commit message: almost done with footprints
Parts:
- U4, U6: footprint (none) -> rov_TCAN_footprint:D0008A-IPC_A
Changed lines of the file:
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@@
 			)
 		)
-		(property "Footprint" ""
+		(property "Footprint" "rov_TCAN_footprint:D0008A-IPC_A"
 			(at 111.76 130.81 0)
 			(hide yes)
@@
 			)
 		)
-		(property "Footprint" ""
+		(property "Footprint" "rov_TCAN_footprint:D0008A-IPC_A"
 			(at 111.76 86.36 0)
 			(hide yes)

Commit message: done with footprints! one more thing for leak sensors
Parts:
- Y1: footprint ECS-120-18-33-JGN-TR:XTAL_ECS-120-18-33-JGN-TR -> rov_ECS_400_18_33_JGN_TR:XTAL_ECS-400-18-33-JGN-TR
- renumbered TP10 to INT0, TP11 to INT1, TP8 to SOF
Changed lines of the file:
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@@
 			)
 		)
-		(property "Footprint" "ECS-120-18-33-JGN-TR:XTAL_ECS-120-18-33-JGN-TR"
+		(property "Footprint" "rov_ECS_400_18_33_JGN_TR:XTAL_ECS-400-18-33-JGN-TR"
 			(at 182.88 43.18 0)
 			(hide yes)
@@
 		(in_pos_files yes)
 		(dnp no)
-		(property "Reference" "TP11"
+		(property "Reference" "INT1"
 			(at 120.65 53.34 90)
 			(show_name no)
@@
 			(project "X19-Pi-Shield-Board"
 				(path "/00000000-0000-0000-0000-000060e6118b/4e72597d-5f14-4a5c-8875-e07f4e1002f7"
-					(reference "TP11")
+					(reference "INT1")
 					(unit 1)
 				)
@@
 		(in_pos_files yes)
 		(dnp no)
-		(property "Reference" "TP8"
+		(property "Reference" "SOF"
 			(at 67.31 40.64 90)
 			(show_name no)
@@
 			(project "X19-Pi-Shield-Board"
 				(path "/00000000-0000-0000-0000-000060e6118b/4e72597d-5f14-4a5c-8875-e07f4e1002f7"
-					(reference "TP8")
+					(reference "SOF")
 					(unit 1)
 				)
@@
 		(in_pos_files yes)
 		(dnp no)
-		(property "Reference" "TP10"
+		(property "Reference" "INT0"
 			(at 120.65 50.8 90)
 			(show_name no)
@@
 			(project "X19-Pi-Shield-Board"
 				(path "/00000000-0000-0000-0000-000060e6118b/4e72597d-5f14-4a5c-8875-e07f4e1002f7"
-					(reference "TP10")
-					(unit 1)
-				)
+					(reference "INT0")
+					(unit 1)
+				)
