File: can.kicad_sch (KiCad schematic)
At the start: 19 parts, among them U4 TCAN1044VDRQ1, U5 MCP2518FDT-E/QBB, U6 TCAN1044VDRQ1, Y1 ECS-400-18-33-JGN-TR

Commit message: footprints COMPLETELY DONE
Parts:
- renumbered SOF to SOF1
Changed lines of the file:
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@@
 		(in_pos_files yes)
 		(dnp no)
-		(property "Reference" "SOF"
+		(property "Reference" "SOF1"
 			(at 67.31 40.64 90)
 			(show_name no)
@@
 			(project "X19-Pi-Shield-Board"
 				(path "/00000000-0000-0000-0000-000060e6118b/4e72597d-5f14-4a5c-8875-e07f4e1002f7"
-					(reference "SOF")
+					(reference "SOF1")
 					(unit 1)
 				)
