File: power.kicad_sch (KiCad schematic)
At the start: 8 parts, among them J9 Conn_01x04_Pin, U1 MIC5504-3.3YM5, U3 INA237AIDGSR

Commit message: changes?
Parts:
- removed J9: Conn_01x04_Pin, symbol Connector:Conn_01x04_Pin
- added J2: Conn_01x02, rov_connectors:0436500200, symbol Connector_Generic:Conn_01x02
Connections:
- net +5V_UNFILT: now also J2.1 (Pin_1)
- net GND: now also C1.2, C2.2, J2.2 (Pin_2)

Commit message: In progress, changed stdby
Connections:
- net +5V_UNFILT renamed +5V_RAW
Other:
- moved on the sheet: J2
Changed lines of the file:
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@@
 	(text "Power IN from Power Slab\n5.2V @9.6A (50W)"
 		(exclude_from_sim no)
-		(at 155.702 38.1 0)
+		(at 127.762 35.56 0)
 		(effects
 			(font
@@
 	(wire
 		(pts
-			(xy 157.48 52.07) (xy 153.67 52.07)
-		)
-		(stroke
-			(width 0)
-			(type default)
-		)
-	)
-	(wire
-		(pts
-			(xy 157.48 53.34) (xy 157.48 52.07)
+			(xy 129.54 49.53) (xy 125.73 49.53)
+		)
+		(stroke
+			(width 0)
+			(type default)
+		)
+	)
+	(wire
+		(pts
+			(xy 129.54 50.8) (xy 129.54 49.53)
 		)
 		(stroke
@@
 	(wire
 		(pts
-			(xy 153.67 49.53) (xy 163.83 49.53)
+			(xy 125.73 46.99) (xy 135.89 46.99)
 		)
 		(stroke
@@
 		)
 	)
-	(label "+5V_UNFILT"
-		(at 163.83 49.53 180)
+	(label "+5V_RAW"
+		(at 135.89 46.99 180)
 		(effects
 			(font
@@
 	(symbol
 		(lib_id "Connector_Generic:Conn_01x02")
-		(at 148.59 49.53 0)
+		(at 120.65 46.99 0)
 		(mirror y)
 		(unit 1)
@@
 		(dnp no)
 		(property "Reference" "J2"
-			(at 148.082 43.688 0)
+			(at 120.142 41.148 0)
 			(show_name no)
 			(do_not_autoplace no)
@@
 		)
 		(property "Value" "Conn_01x02"
-			(at 152.654 45.72 0)
+			(at 124.714 43.18 0)
 			(show_name no)
 			(do_not_autoplace no)
@@
 		)
 		(property "Footprint" "rov_connectors:0436500200"
-			(at 148.59 49.53 0)
+			(at 120.65 46.99 0)
 			(hide yes)
 			(show_name no)
@@
 		)
 		(property "Datasheet" ""
-			(at 148.59 49.53 0)
+			(at 120.65 46.99 0)
 			(hide yes)
 			(show_name no)
@@
 		)
 		(property "Description" "Generic connector, single row, 01x02, script generated (kicad-library-utils/schlib/autogen/connector/)"
-			(at 148.59 49.53 0)
+			(at 120.65 46.99 0)
 			(hide yes)
 			(show_name no)
@@
 			)
 		)
-		(property "Value" "+5V_UNFILT"
-			(at 91.44 27.94 0)
-			(show_name no)
-			(do_not_autoplace no)
-			(effects
-				(font
-					(size 1.27 1.27)
-				)
+		(property "Value" "+5V_RAW"
+			(at 93.98 31.7499 0)
+			(show_name no)
+			(do_not_autoplace no)
+			(effects
+				(font
+					(size 1.27 1.27)
+				)
+				(justify left)
 			)
 		)
@@
 	(symbol
 		(lib_id "power:GND")
-		(at 157.48 53.34 0)
+		(at 129.54 50.8 0)
 		(unit 1)
 		(body_style 1)
@@
 		(dnp no)
 		(property "Reference" "#PWR08"
-			(at 157.48 59.69 0)
+			(at 129.54 57.15 0)
 			(hide yes)
 			(show_name no)
@@
 		)
 		(property "Value" "GND"
-			(at 161.29 55.118 0)
+			(at 133.35 52.578 0)
 			(show_name no)
 			(do_not_autoplace no)
@@
 		)
 		(property "Footprint" ""
-			(at 157.48 53.34 0)
+			(at 129.54 50.8 0)
 			(hide yes)
 			(show_name no)
@@
 		)
 		(property "Datasheet" ""
-			(at 157.48 53.34 0)
+			(at 129.54 50.8 0)
 			(hide yes)
 			(show_name no)
@@
 		)
 		(property "Description" "Power symbol creates a global label with name \"GND\" , ground"
-			(at 157.48 53.34 0)
-			(hide yes)
-			(show_name no)
+			(at 129.54 50.8 0)
+			(hide yes)
+			(show_name no)

Commit message: Relatively final changes
Parts:
- added C16: 47uF, symbol Device:C
- added C18: 100n, symbol Device:C
- C1, C2: value 1uF -> 1u
- C5: value 0.1uF -> 100n
Connections:
- net +3.3V: now also C5.1, U3.6 (VS)
- net GND: now also C16.2, C18.2
- net +5V renamed +5.1V
- net +5.1V: no longer C5.1, U3.6 (VS)
- net +5V_RAW renamed +5.1V_RAW
- net +5.1V_RAW: now also C16.1, C18.1
Other:
- moved on the sheet: C1, C2, J2, R1, R4, U1, U3

Commit message: Some minor changes
Connections:
- net GPIO_ALERT renamed ALERT_5.1V
Changed lines of the file:
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@@
+	)
+	(junction
+		(at 146.05 90.17)
+		(diameter 0)
+		(color 0 0 0 0)
+	)
+	(junction
+		(at 134.62 125.73)
+		(diameter 0)
+		(color 0 0 0 0)
 	)
 	(junction
@@
 		(color 0 0 0 0)
 	)
-	(junction
-		(at 146.05 90.17)
-		(diameter 0)
-		(color 0 0 0 0)
-	)
-	(junction
-		(at 134.62 125.73)
-		(diameter 0)
-		(color 0 0 0 0)
-	)
 	(wire
 		(pts
@@
 		(pts
 			(xy 143.51 92.71) (xy 146.05 92.71)
+		)
+		(stroke
+			(width 0)
+			(type default)
+		)
+	)
+	(wire
+		(pts
+			(xy 147.32 93.98) (xy 147.32 95.25)
 		)
 		(stroke
@@
 		(effects
 			(font
-				(size 0.889 0.889)
+				(size 1.27 1.27)
 			)
 			(justify right)
 		)
 		(property "Intersheetrefs" "${INTERSHEET_REFS}"
-			(at 77.4894 100.33 0)
+			(at 73.1434 100.33 0)
 			(hide yes)
 			(show_name no)
@@
 		(effects
 			(font
-				(size 0.889 0.889)
+				(size 1.27 1.27)
 			)
 			(justify right)
 		)
 		(property "Intersheetrefs" "${INTERSHEET_REFS}"
-			(at 77.4471 95.25 0)
+			(at 73.0829 95.25 0)
 			(hide yes)
 			(show_name no)
@@
 		)
 	)
-	(global_label "GPIO_ALERT"
+	(global_label "ALERT_5.1V"
 		(shape input)
 		(at 88.9 90.17 180)
@@
 		(effects
 			(font
-				(size 0.889 0.889)
+				(size 1.27 1.27)
 			)
 			(justify right)
 		)
 		(property "Intersheetrefs" "${INTERSHEET_REFS}"
-			(at 79.6062 90.17 0)
+			(at 75.9857 90.17 0)
 			(hide yes)
 			(show_name no)
@@
 	(symbol
 		(lib_id "power:+5V")
-		(at 147.32 95.25 0)
+		(at 147.32 93.98 0)
 		(unit 1)
 		(body_style 1)
@@
 		(dnp no)
 		(property "Reference" "#PWR017"
-			(at 147.32 99.06 0)
+			(at 147.32 97.79 0)
 			(hide yes)
 			(show_name no)
@@
 		)
 		(property "Value" "+3.3V"
-			(at 151.13 93.98 0)
+			(at 151.13 92.71 0)
 			(show_name no)
 			(do_not_autoplace no)
@@
 		)
 		(property "Footprint" ""
-			(at 147.32 95.25 0)
+			(at 147.32 93.98 0)
 			(hide yes)
 			(show_name no)
@@
 		)
 		(property "Datasheet" ""
-			(at 147.32 95.25 0)
+			(at 147.32 93.98 0)
 			(hide yes)
 			(show_name no)
@@
 		)
 		(property "Description" "Power symbol creates a global label with name \"+5V\""
-			(at 147.32 95.25 0)
+			(at 147.32 93.98 0)
 			(hide yes)
 			(show_name no)
@@
 		)
 		(property "Value" "GND"
-			(at 104.648 87.122 0)
+			(at 97.79 87.63 0)
 			(show_name no)
 			(do_not_autoplace no)
@@
 		(dnp no)
 		(property "Reference" "R1"
-			(at 141.478 87.884 0)
+			(at 142.24 87.63 0)
 			(show_name no)
 			(do_not_autoplace no)
@@
 		)
 		(property "Value" "1m"
-			(at 141.224 86.106 0)
+			(at 141.986 85.852 0)
 			(show_name no)
 			(do_not_autoplace no)
@@
 			(effects
 				(font
-					(size 0.889 0.889)
-				)
-			)
+					(size 1.27 1.27)
+				)
+			)

Commit message: updated footprints
Parts:
- R1: footprint D0008A-IPC_A -> (none)
- U3: footprint VSSOP_IDGSR_TEX -> (none)
Changed lines of the file:
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@@
 			)
 		)
-		(property "Footprint" "D0008A-IPC_A"
+		(property "Footprint" ""
 			(at 146.05 86.36 0)
 			(hide yes)
@@
 			)
 		)
-		(property "Footprint" "VSSOP_IDGSR_TEX"
+		(property "Footprint" ""
 			(at 102.87 86.36 0)
 			(hide yes)

Commit message: added footprints
Parts:
- C16: footprint (none) -> Capacitor_SMD:C_0805_2012Metric_Pad1.18x1.45mm_HandSolder
- C18, C5: footprint (none) -> Capacitor_SMD:C_0603_1608Metric_Pad1.08x0.95mm_HandSolder
- R1: footprint (none) -> Resistor_SMD:R_2512_6332Metric_Pad1.40x3.35mm_HandSolder
- R4: footprint (none) -> Resistor_SMD:R_0603_1608Metric_Pad0.98x0.95mm_HandSolder
Changed lines of the file:
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@@
 			)
 		)
-		(property "Footprint" ""
+		(property "Footprint" "Capacitor_SMD:C_0603_1608Metric_Pad1.08x0.95mm_HandSolder"
 			(at 213.0552 96.52 0)
 			(hide yes)
@@
 		)
 		(property "Description" "Unpolarized capacitor"
+			(at 212.09 92.71 0)
+			(hide yes)
+			(show_name no)
+			(do_not_autoplace no)
+			(effects
+				(font
+					(size 1.27 1.27)
+				)
+			)
+		)
+		(property "digikey" ""
 			(at 212.09 92.71 0)
 			(hide yes)
@@
 			)
 		)
-		(property "Footprint" ""
+		(property "Footprint" "Capacitor_SMD:C_0603_1608Metric_Pad1.08x0.95mm_HandSolder"
 			(at 148.2852 102.87 0)
 			(hide yes)
@@
 		)
 		(property "Description" "Unpolarized capacitor"
+			(at 147.32 99.06 0)
+			(hide yes)
+			(show_name no)
+			(do_not_autoplace no)
+			(effects
+				(font
+					(size 1.27 1.27)
+				)
+			)
+		)
+		(property "digikey" ""
 			(at 147.32 99.06 0)
 			(hide yes)
@@
 			)
 		)
-		(property "Footprint" ""
+		(property "Footprint" "Capacitor_SMD:C_0805_2012Metric_Pad1.18x1.45mm_HandSolder"
 			(at 199.0852 96.52 0)
 			(hide yes)
@@
 		)
 		(property "Description" "Unpolarized capacitor"
+			(at 198.12 92.71 0)
+			(hide yes)
+			(show_name no)
+			(do_not_autoplace no)
+			(effects
+				(font
+					(size 1.27 1.27)
+				)
+			)
+		)
+		(property "digikey" ""
 			(at 198.12 92.71 0)
 			(hide yes)
@@
 			)
 		)
+		(property "digikey" ""
+			(at 175.26 91.44 0)
+			(hide yes)
+			(show_name no)
+			(do_not_autoplace no)
+			(effects
+				(font
+					(size 1.27 1.27)
+				)
+			)
+		)
 		(pin "2"
 		)
@@
 			)
 		)
-		(property "Footprint" ""
+		(property "Footprint" "Resistor_SMD:R_2512_6332Metric_Pad1.40x3.35mm_HandSolder"
 			(at 146.05 86.36 0)
 			(hide yes)
@@
 		)
 		(property "Description" "Resistor, small US symbol"
+			(at 146.05 86.36 0)
+			(hide yes)
+			(show_name no)
+			(do_not_autoplace no)
+			(effects
+				(font
+					(size 1.27 1.27)
+				)
+			)
+		)
+		(property "digikey" ""
 			(at 146.05 86.36 0)
 			(hide yes)
@@
 			)
 		)
+		(property "digikey" ""
+			(at 93.98 130.81 0)
+			(hide yes)
+			(show_name no)
+			(do_not_autoplace no)
+			(effects
+				(font
+					(size 1.27 1.27)
+				)
+			)
+		)
 		(pin "2"
 		)
@@
 			)
 		)
+		(property "digikey" ""
+			(at 102.87 86.36 0)
+			(hide yes)
+			(show_name no)
+			(do_not_autoplace no)
+			(effects
+				(font
+					(size 1.27 1.27)
+				)
+			)
+		)
 		(pin "9"
 		)
@@
 			)
 		)
+		(property "digikey" ""
+			(at 134.62 130.81 0)
+			(hide yes)
+			(show_name no)
+			(do_not_autoplace no)
+			(effects
+				(font
+					(size 1.27 1.27)
+				)
+			)
+		)
 		(pin "2"
 		)
@@
 			)
 		)
-		(property "Footprint" ""
+		(property "Footprint" "Resistor_SMD:R_0603_1608Metric_Pad0.98x0.95mm_HandSolder"
 			(at 90.17 82.55 0)
 			(hide yes)
@@
 		)
 		(property "Description" "Resistor, small US symbol"
+			(at 90.17 82.55 0)
+			(hide yes)
+			(show_name no)
+			(do_not_autoplace no)
+			(effects
+				(font
+					(size 1.27 1.27)
+				)
+			)
+		)
+		(property "digikey" ""
 			(at 90.17 82.55 0)
 			(hide yes)
@@
 			(at 114.3 128.27 0)
 			(hide yes)
+			(show_name no)
+			(do_not_autoplace no)
+			(effects
+				(font
+					(size 1.27 1.27)
+				)
+			)
+		)
+		(property "digikey" ""
+			(at 114.3 128.27 0)
+			(hide yes)

Commit message: almost done with footprints
Parts:
- U3: footprint (none) -> rov_INA_footprint:VSSOP_IDGSR_TEX-M
Changed lines of the file:
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@@
 			)
 		)
-		(property "Footprint" ""
+		(property "Footprint" "rov_INA_footprint:VSSOP_IDGSR_TEX-M"
 			(at 102.87 86.36 0)
 			(hide yes)

Commit message: done with footprints! one more thing for leak sensors
Parts:
- C1, C2: footprint Package_SO:SOIC-8_3.9x4.9mm_P1.27mm -> Capacitor_SMD:C_0603_1608Metric_Pad1.08x0.95mm_HandSolder
- C16: footprint Capacitor_SMD:C_0805_2012Metric_Pad1.18x1.45mm_HandSolder -> Capacitor_SMD:C_1210_3225Metric_Pad1.33x2.70mm_HandSolder
- J2: footprint rov_connectors:0436500200 -> rov_conn_436500200:CONN_SD-43650-001_02_MOL
- R1: footprint Resistor_SMD:R_2512_6332Metric_Pad1.40x3.35mm_HandSolder -> Resistor_SMD:R_1206_3216Metric_Pad1.30x1.75mm_HandSolder
Changed lines of the file:
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@@
 			)
 		)
-		(property "Footprint" "Capacitor_SMD:C_0805_2012Metric_Pad1.18x1.45mm_HandSolder"
+		(property "Footprint" "Capacitor_SMD:C_1210_3225Metric_Pad1.33x2.70mm_HandSolder"
 			(at 199.0852 96.52 0)
 			(hide yes)
@@
 			)
 		)
-		(property "Footprint" "rov_connectors:0436500200"
+		(property "Footprint" "rov_conn_436500200:CONN_SD-43650-001_02_MOL"
 			(at 175.26 91.44 0)
 			(hide yes)
@@
 			)
 		)
-		(property "Footprint" "Resistor_SMD:R_2512_6332Metric_Pad1.40x3.35mm_HandSolder"
+		(property "Footprint" "Resistor_SMD:R_1206_3216Metric_Pad1.30x1.75mm_HandSolder"
 			(at 146.05 86.36 0)
 			(hide yes)
@@
 			)
 		)
-		(property "Footprint" "Package_SO:SOIC-8_3.9x4.9mm_P1.27mm"
+		(property "Footprint" "Capacitor_SMD:C_0603_1608Metric_Pad1.08x0.95mm_HandSolder"
 			(at 94.9452 134.62 0)
 			(hide yes)
@@
 			)
 		)
-		(property "Footprint" "Package_SO:SOIC-8_3.9x4.9mm_P1.27mm"
+		(property "Footprint" "Capacitor_SMD:C_0603_1608Metric_Pad1.08x0.95mm_HandSolder"
 			(at 135.5852 134.62 0)
 			(hide yes)
